Commit message: Fixed world frame issues for checking 'top' of object and remade geometry extraction node to properly get the top and get a polygon using cv instead of convexhull

File: top_surface_enviornment/urdf/camera.urdf (robot description, URDF)
Before this commit: robot camera, 4 links, 3 joints
Links:
- removed link world
- link camera_link: mass 1e-5 -> 0.2
Joints:
- removed joint world_to_base
